File: 2013/pcb/servoDriver/servoDrv.brd (EAGLE design)
At the start: 19.4 x 16.4 mm, 9 parts, among them X1 22-23-2041

Commit message: Pieniä muutoksia servo pcb:hen Servojen H-sillan manuaali lisätty
Parts:
- U1: value (none) -> SI9986DY-T1-E3
- X2: value (none) -> MOTOR
Connections:
- net VCC renamed VDD
Changed lines of the file:
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@@
 </autorouter>
 <elements>
-<element name="U1" library="vishay_motor" package="SOIC127P600X175-8N" value="" x="11.43" y="7.82" rot="MR180">
+<element name="U1" library="vishay_motor" package="SOIC127P600X175-8N" value="SI9986DY-T1-E3" x="11.43" y="7.82" rot="MR180">
 <attribute name="PACKAGE" value="SOIC-8" x="40.64" y="11.63" size="1.778" layer="28" rot="MR180" display="off"/>
 <attribute name="OC_NEWARK" value="06J8287" x="40.64" y="11.63" size="1.778" layer="28" rot="MR180" display="off"/>
@@
 <attribute name="OC_FARNELL" value="1462920" x="-4.60984375" y="-11.4499375" size="1.778" layer="27" rot="R270" display="off"/>
 </element>
-<element name="X2" library="con-ptr500" package="AK500/2" value="" x="17.11" y="8.22" rot="R90">
+<element name="X2" library="con-ptr500" package="AK500/2" value="MOTOR" x="17.11" y="8.22" rot="R90">
 <attribute name="OC_NEWARK" value="unknown" x="31.08" y="24.73" size="1.778" layer="27" rot="R90" display="off"/>
 <attribute name="MPN" value="" x="31.08" y="24.73" size="1.778" layer="27" rot="R90" display="off"/>
@@
 </elements>
 <signals>
-<signal name="VCC">
+<signal name="VDD">
 <contactref element="U1" pad="3"/>
 <contactref element="C1" pad="1"/>
