File: 2013/pcb/servoDriver/servoDrv.sch (EAGLE design)
At the start: 9 parts, among them X1 22-23-2041

Commit message: Muutettu servoDriver pcb yksipuoleiseksi
Parts:
- RIN_A, RIN_B: device resistor:R-EU_R0805 -> resistor2:R-EU_0207/10
Changed lines of the file:
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@@
 <?xml version="1.0" encoding="utf-8"?>
 <!DOCTYPE eagle SYSTEM "eagle.dtd">
-<eagle version="6.5.0">
+<eagle version="6.4">
 <drawing>
 <settings>
@@
 <grid distance="0.1" unitdist="inch" unit="inch" style="lines" multiple="1" display="no" altdistance="0.01" altunitdist="inch" altunit="inch"/>
 <layers>
-<layer number="1" name="Top" color="4" fill="1" visible="no" active="no"/>
-<layer number="16" name="Bottom" color="1" fill="1" visible="no" active="no"/>
-<layer number="17" name="Pads" color="2" fill="1" visible="no" active="no"/>
-<layer number="18" name="Vias" color="2" fill="1" visible="no" active="no"/>
-<layer number="19" name="Unrouted" color="6" fill="1" visible="no" active="no"/>
-<layer number="20" name="Dimension" color="15" fill="1" visible="no" active="no"/>
-<layer number="21" name="tPlace" color="7" fill="1" visible="no" active="no"/>
-<layer number="22" name="bPlace" color="7" fill="1" visible="no" active="no"/>
-<layer number="23" name="tOrigins" color="15" fill="1" visible="no" active="no"/>
-<layer number="24" name="bOrigins" color="15" fill="1" visible="no" active="no"/>
-<layer number="25" name="tNames" color="7" fill="1" visible="no" active="no"/>
-<layer number="26" name="bNames" color="7" fill="1" visible="no" active="no"/>
-<layer number="27" name="tValues" color="7" fill="1" visible="no" active="no"/>
-<layer number="28" name="bValues" color="7" fill="1" visible="no" active="no"/>
+<layer number="1" name="Top" color="4" fill="1" visible="yes" active="no"/>
+<layer number="16" name="Bottom" color="1" fill="1" visible="yes" active="no"/>
+<layer number="17" name="Pads" color="2" fill="1" visible="yes" active="no"/>
+<layer number="18" name="Vias" color="2" fill="1" visible="yes" active="no"/>
+<layer number="19" name="Unrouted" color="6" fill="1" visible="yes" active="no"/>
+<layer number="20" name="Dimension" color="15" fill="1" visible="yes" active="no"/>
+<layer number="21" name="tPlace" color="7" fill="1" visible="yes" active="no"/>
+<layer number="22" name="bPlace" color="7" fill="1" visible="yes" active="no"/>
+<layer number="23" name="tOrigins" color="15" fill="1" visible="yes" active="no"/>
+<layer number="24" name="bOrigins" color="15" fill="1" visible="yes" active="no"/>
+<layer number="25" name="tNames" color="7" fill="1" visible="yes" active="no"/>
+<layer number="26" name="bNames" color="7" fill="1" visible="yes" active="no"/>
+<layer number="27" name="tValues" color="7" fill="1" visible="yes" active="no"/>
+<layer number="28" name="bValues" color="7" fill="1" visible="yes" active="no"/>
 <layer number="29" name="tStop" color="7" fill="3" visible="no" active="no"/>
 <layer number="30" name="bStop" color="7" fill="6" visible="no" active="no"/>
@@
 <layer number="35" name="tGlue" color="7" fill="4" visible="no" active="no"/>
 <layer number="36" name="bGlue" color="7" fill="5" visible="no" active="no"/>
-<layer number="37" name="tTest" color="7" fill="1" visible="no" active="no"/>
-<layer number="38" name="bTest" color="7" fill="1" visible="no" active="no"/>
+<layer number="37" name="tTest" color="7" fill="1" visible="yes" active="no"/>
+<layer number="38" name="bTest" color="7" fill="1" visible="yes" active="no"/>
 <layer number="39" name="tKeepout" color="4" fill="11" visible="no" active="no"/>
 <layer number="40" name="bKeepout" color="1" fill="11" visible="no" active="no"/>
@@
 <layer number="44" name="Drills" color="7" fill="1" visible="no" active="no"/>
 <layer number="45" name="Holes" color="7" fill="1" visible="no" active="no"/>
-<layer number="46" name="Milling" color="3" fill="1" visible="no" active="no"/>
-<layer number="47" name="Measures" color="7" fill="1" visible="no" active="no"/>
-<layer number="48" name="Document" color="7" fill="1" visible="no" active="no"/>
-<layer number="49" name="Reference" color="7" fill="1" visible="no" active="no"/>
-<layer number="51" name="tDocu" color="7" fill="1" visible="no" active="no"/>
-<layer number="52" name="bDocu" color="7" fill="1" visible="no" active="no"/>
+<layer number="46" name="Milling" color="3" fill="1" visible="yes" active="no"/>
+<layer number="47" name="Measures" color="7" fill="1" visible="yes" active="no"/>
+<layer number="48" name="Document" color="7" fill="1" visible="yes" active="no"/>
+<layer number="49" name="Reference" color="7" fill="1" visible="yes" active="no"/>
+<layer number="51" name="tDocu" color="7" fill="1" visible="yes" active="no"/>
+<layer number="52" name="bDocu" color="7" fill="1" visible="yes" active="no"/>
 <layer number="91" name="Nets" color="2" fill="1" visible="yes" active="yes"/>
 <layer number="92" name="Busses" color="1" fill="1" visible="yes" active="yes"/>
@@
 <part name="X1" library="con-molex" deviceset="22-23-2041" device=""/>
 <part name="X2" library="con-ptr500" deviceset="AK500/2" device=""/>
-<part name="RIN_A" library="resistor" deviceset="R-EU_" device="R0805" value="100"/>
-<part name="RIN_B" library="resistor" deviceset="R-EU_" device="R0805" value="100"/>
+<part name="RIN_A" library="resistor2" deviceset="R-EU_" device="0207/10" value="100"/>
+<part name="RIN_B" library="resistor2" deviceset="R-EU_" device="0207/10" value="100"/>
 <part name="C1" library="resistor" deviceset="C-EU" device="C0805" value="100n"/>
 <part name="C2" library="resistor" deviceset="C-EU" device="C0805" value="1u"/>

Commit message: Pieniä muutoksia servo pcb:hen Servojen H-sillan manuaali lisätty
Parts:
- U1: value (none) -> SI9986DY-T1-E3
- X2: value (none) -> MOTOR
Connections:
- net VCC renamed VDD
Other:
- moved on the sheet: C2
Changed lines of the file:
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@@
 </classes>
 <parts>
-<part name="U1" library="vishay_motor" deviceset="SI9986DY-T1-E3" device=""/>
-<part name="P+1" library="supply1" deviceset="VCC" device=""/>
+<part name="U1" library="vishay_motor" deviceset="SI9986DY-T1-E3" device="" value="SI9986DY-T1-E3"/>
+<part name="P+1" library="supply1" deviceset="VDD" device=""/>
 <part name="GND1" library="supply1" deviceset="GND" device=""/>
 <part name="X1" library="con-molex" deviceset="22-23-2041" device=""/>
-<part name="X2" library="con-ptr500" deviceset="AK500/2" device=""/>
+<part name="X2" library="con-ptr500" deviceset="AK500/2" device="" value="MOTOR"/>
 <part name="RIN_A" library="resistor2" deviceset="R-EU_" device="0207/10" value="100"/>
 <part name="RIN_B" library="resistor2" deviceset="R-EU_" device="0207/10" value="100"/>
 <part name="C1" library="resistor" deviceset="C-EU" device="C0805" value="100n"/>
 <part name="C2" library="resistor" deviceset="C-EU" device="C0805" value="1u"/>
-<part name="P+2" library="supply1" deviceset="VCC" device=""/>
+<part name="P+2" library="supply1" deviceset="VDD" device=""/>
 <part name="GND2" library="supply1" deviceset="GND" device=""/>
 <part name="D1" library="diode" deviceset="DIODE-" device="SOD123" value="PTVS6V0S1UR"/>
@@
 <instances>
 <instance part="U1" gate="A" x="45.72" y="60.96"/>
-<instance part="P+1" gate="VCC" x="7.62" y="91.44"/>
+<instance part="P+1" gate="G$1" x="7.62" y="91.44"/>
 <instance part="GND1" gate="1" x="-12.7" y="33.02"/>
 <instance part="X1" gate="-1" x="-20.32" y="60.96" rot="MR0"/>
@@
 <instance part="RIN_B" gate="G$1" x="12.7" y="60.96"/>
 <instance part="C1" gate="G$1" x="93.98" y="66.04"/>
-<instance part="C2" gate="G$1" x="101.6" y="66.04"/>
-<instance part="P+2" gate="VCC" x="93.98" y="81.28"/>
+<instance part="C2" gate="G$1" x="106.68" y="66.04"/>
+<instance part="P+2" gate="G$1" x="93.98" y="81.28"/>
 <instance part="GND2" gate="1" x="96.52" y="38.1"/>
 <instance part="D1" gate="G$1" x="-5.08" y="48.26" rot="R90"/>
@@
 </busses>
 <nets>
-<net name="VCC" class="0">
+<net name="VDD" class="0">
 <segment>
-<pinref part="P+1" gate="VCC" pin="VCC"/>
+<pinref part="P+1" gate="G$1" pin="VDD"/>
 <wire x1="7.62" y1="68.58" x2="7.62" y2="78.74" width="0.1524" layer="91"/>
 <pinref part="U1" gate="A" pin="VDD"/>
@@
 <pinref part="X1" gate="-2" pin="S"/>
 <wire x1="-17.78" y1="68.58" x2="7.62" y2="68.58" width="0.1524" layer="91"/>
+<junction x="7.62" y="78.74"/>
 </segment>
 <segment>
-<pinref part="P+2" gate="VCC" pin="VCC"/>
+<pinref part="P+2" gate="G$1" pin="VDD"/>
 <pinref part="C1" gate="G$1" pin="1"/>
-<wire x1="93.98" y1="78.74" x2="93.98" y2="76.2" width="0.1524" layer="91"/>
 <pinref part="C2" gate="G$1" pin="1"/>
-<wire x1="101.6" y1="68.58" x2="93.98" y2="68.58" width="0.1524" layer="91"/>
-<wire x1="93.98" y1="68.58" x2="93.98" y2="76.2" width="0.1524" layer="91"/>
+<wire x1="106.68" y1="68.58" x2="93.98" y2="68.58" width="0.1524" layer="91"/>
+<wire x1="93.98" y1="68.58" x2="93.98" y2="78.74" width="0.1524" layer="91"/>
+<junction x="93.98" y="68.58"/>
 </segment>
 </net>
@@
 <pinref part="C1" gate="G$1" pin="2"/>
 <wire x1="96.52" y1="40.64" x2="93.98" y2="40.64" width="0.1524" layer="91"/>
-<wire x1="93.98" y1="40.64" x2="93.98" y2="55.88" width="0.1524" layer="91"/>
+<wire x1="93.98" y1="40.64" x2="93.98" y2="60.96" width="0.1524" layer="91"/>
 <pinref part="C2" gate="G$1" pin="2"/>
-<wire x1="101.6" y1="60.96" x2="93.98" y2="60.96" width="0.1524" layer="91"/>
-<wire x1="93.98" y1="60.96" x2="93.98" y2="55.88" width="0.1524" layer="91"/>
+<wire x1="106.68" y1="60.96" x2="93.98" y2="60.96" width="0.1524" layer="91"/>
+<junction x="93.98" y="60.96"/>
 </segment>
 <segment>
@@
 <wire x1="15.24" y1="53.34" x2="15.24" y2="33.02" width="0.1524" layer="91"/>
 <wire x1="27.94" y1="53.34" x2="15.24" y2="53.34" width="0.1524" layer="91"/>
+<junction x="15.24" y="53.34"/>
 </segment>
 <segment>
@@
 <wire x1="0" y1="60.96" x2="7.62" y2="60.96" width="0.1524" layer="91"/>
 <wire x1="0" y1="50.8" x2="0" y2="60.96" width="0.1524" layer="91"/>
+<junction x="0" y="60.96"/>
 </segment>
 </net>
@@
 <wire x1="-5.08" y1="66.04" x2="7.62" y2="66.04" width="0.1524" layer="91"/>
 <wire x1="-5.08" y1="50.8" x2="-5.08" y2="66.04" width="0.1524" layer="91"/>
+<junction x="-5.08" y="66.04"/>
 </segment>
 </net>
